Commit message: Added models for xarm7 Gazebo simulation and changed code to work with it

File: xarm_description/urdf/camera/realsense_d435i.urdf.xacro (robot description, xacro)
@@ -15,4 +15,7 @@
         origin_rpy="0 0 0" />
     </link>
+    <gazebo reference="${prefix}link_eef">
+      <material>Gazebo/Indigo</material>
+    </gazebo>
     <xacro:if value="${add_d435i_links}">
       <link name="${prefix}camera_link"></link>

File: xarm_description/urdf/common/common.material.xacro (robot description, xacro)
@@ -6,5 +6,5 @@
     </material>
     <material name="${prefix}Red">
-      <color rgba="0.8 0.0 0.0 1.0"/>
+      <color rgba="0.8 0.5 0.5 1.0"/>
     </material>
     <material name="${prefix}White">
@@ -14,4 +14,11 @@
       <color rgba="0.753 0.753 0.753 1.0"/>
     </material>
+    <material name="${prefix}Grey">
+      <color rgba="0.5 0.5 0.5 1.0"/>
+    </material>
+    <!-- ✅ New Industrial Blue -->
+    <material name="${prefix}IndustrialBlue">
+      <color rgba="0.2 0.3 0.5 1.0"/>
+    </material>
   </xacro:macro>
 </robot>

File: xarm_description/urdf/vacuum_gripper/xarm_vacuum_gripper.urdf.xacro (robot description, xacro)
@@ -9,4 +9,7 @@
       </joint>
     </xacro:unless>
+    <gazebo reference="${prefix}xarm_vacuum_gripper_link">
+      <material>Gazebo/Orange</material>
+    </gazebo>
     <link name="${prefix}xarm_vacuum_gripper_link">
       <inertial>

File: xarm_description/urdf/xarm7/xarm7.gazebo.xacro (robot description, xacro)
@@ -2,27 +2,36 @@
 <robot xmlns:xacro="http://ros.org/wiki/xacro">
   <xacro:macro name="xarm7_gazebo" params="prefix">
+    <!-- Base and Arm -->
     <gazebo reference="${prefix}link_base">
       <selfCollide>true</selfCollide>
+      <material>Gazebo/Grey</material>
     </gazebo>
     <gazebo reference="${prefix}link1">
       <selfCollide>true</selfCollide>
+      <material>Gazebo/Grey</material>
     </gazebo>
     <gazebo reference="${prefix}link2">
       <selfCollide>true</selfCollide>
+      <material>Gazebo/Grey</material>
     </gazebo>
     <gazebo reference="${prefix}link3">
       <selfCollide>true</selfCollide>
+      <material>Gazebo/Grey</material>
     </gazebo>
     <gazebo reference="${prefix}link4">
       <selfCollide>true</selfCollide>
+      <material>Gazebo/Grey</material>
     </gazebo>
     <gazebo reference="${prefix}link5">
       <selfCollide>true</selfCollide>
+      <material>Gazebo/Grey</material>
     </gazebo>
     <gazebo reference="${prefix}link6">
       <selfCollide>true</selfCollide>
+      <material>Gazebo/Grey</material>
     </gazebo>
     <gazebo reference="${prefix}link7">
       <selfCollide>true</selfCollide>
+      <material>Gazebo/Grey</material>
     </gazebo>
   </xacro:macro>

File: xarm_moveit_config/srdf/_xarm7_macro.srdf.xacro (robot description, xacro)
@@ -67,12 +67,4 @@
       <joint name="${prefix}joint7" value="-0.025441950871051056" />
     </group_state>
-    look:
-  - 0.1388548331359134
-  - -0.35411523916076515
-  - -0.17444431215925871
-  - 1.4426785833000872
-  - -0.061715033311549483
-  - 1.7915080917332666
-  - -0.025441950871051056
     <group_state name="pick_pre" group="${prefix}xarm7">
       <joint name="${prefix}joint1" value="0.19919301702224512" />
@@ -102,5 +94,5 @@
       <joint name="${prefix}joint7" value="-5.5301690339737419e-05" />
     </group_state>
-    <group_state name="_post" group="${prefix}xarm7">
+    <group_state name="drop_post" group="${prefix}xarm7">
       <joint name="${prefix}joint1" value="0.034168209390873727" />
       <joint name="${prefix}joint2" value="0.27173424338337426" />
@@ -138,12 +130,48 @@
       <joint name="${prefix}joint7" value="-0.092139458728333956" />
     </group_state>
-    <group_state name="look1" group="${prefix}xarm7">
-      <joint name="${prefix}joint1" value="0.26049781339689471" />
-      <joint name="${prefix}joint2" value="0.71173226837173598" />
-      <joint name="${prefix}joint3" value="0.092265167922493063" />
-      <joint name="${prefix}joint4" value="1.1172871190565097" />
-      <joint name="${prefix}joint5" value="0.26840659938472733" />
-      <joint name="${prefix}joint6" value="-1.2196054769755964" />
-      <joint name="${prefix}joint7" value="-0.20052051080472882" />
+    <group_state name="hi1" group="${prefix}xarm7">
+      <joint name="${prefix}joint1" value="0.15537082420215143" />
+      <joint name="${prefix}joint2" value="-0.57023563298973912" />
+      <joint name="${prefix}joint3" value="-0.32224262043483787" />
+      <joint name="${prefix}joint4" value="1.4348493236202611" />
+      <joint name="${prefix}joint5" value="0.11975100198797506" />
+      <joint name="${prefix}joint6" value="0.66577686218844612" />
+      <joint name="${prefix}joint7" value="-0.28959232208729446" />
+    </group_state>
+    <group_state name="hi2" group="${prefix}xarm7">
+      <joint name="${prefix}joint1" value="0.5850001582454567" />
+      <joint name="${prefix}joint2" value="-0.36624042681323221" />
+      <joint name="${prefix}joint3" value="-0.59730367237416182" />
+      <joint name="${prefix}joint4" value="1.2838524230455413" />
+      <joint name="${prefix}joint5" value="0.59301778808555561" />
+      <joint name="${prefix}joint6" value="-0.021139437939052819" />
+      <joint name="${prefix}joint7" value="-0.79610833776672507" />
+    </group_state>
+    <group_state name="hi3" group="${prefix}xarm7">
+      <joint name="${prefix}joint1" value="0.65592591966536506" />
+      <joint name="${prefix}joint2" value="-0.32931007368005272" />
+      <joint name="${prefix}joint3" value="-0.66285977526225803" />
+      <joint name="${prefix}joint4" value="1.3277492270531326" />
+      <joint name="${prefix}joint5" value="0.61586256867169009" />
+      <joint name="${prefix}joint6" value="-0.021629479047719613" />
+      <joint name="${prefix}joint7" value="-0.81654617572214772" />
+    </group_state>
+    <group_state name="hi4" group="${prefix}xarm7">
+      <joint name="${prefix}joint1" value="0.061876297560076843" />
+      <joint name="${prefix}joint2" value="-0.88977736339482671" />
+      <joint name="${prefix}joint3" value="-0.25310785661261548" />
+      <joint name="${prefix}joint4" value="1.243578324593245" />
+      <joint name="${prefix}joint5" value="0.20338356412763137" />
+      <joint name="${prefix}joint6" value="0.54117266377276074" />
+      <joint name="${prefix}joint7" value="-0.36829799173944444" />
+    </group_state>
+    <group_state name="himain" group="${prefix}xarm7">
+      <joint name="${prefix}joint1" value="-6.0444591986730245e-05" />
+      <joint name="${prefix}joint2" value="-1.0148089645448195" />
+      <joint name="${prefix}joint3" value="-3.7113203106287074e-06" />
+      <joint name="${prefix}joint4" value="0.33800962290575853" />
+      <joint name="${prefix}joint5" value="1.0089107007615894e-05" />
+      <joint name="${prefix}joint6" value="1.3528371032180022" />
+      <joint name="${prefix}joint7" value="9.1350534141554363e-06" />
     </group_state>
     <!-- gripper -->
